File: HW/MarstekMonitor.kicad_sch (KiCad schematic)
At the start: 10 parts, among them J1 Conn_01x06_Socket

Commit message: PCB layout updated
Fixed wrong GPIO pin for RX
Connections:
- net RXD: now also TTGO1.19 (GPIO15); no longer TTGO1.21 (GPIO12)
Changed lines of the file:
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@@
-	)
-	(no_connect
-		(at 127 77.47)
 	)
 	(no_connect
@@
 	)
 	(no_connect
+		(at 127 82.55)
+	)
+	(no_connect
 		(at 154.94 77.47)
 	)
@@
 	(wire
 		(pts
-			(xy 119.38 82.55) (xy 127 82.55)
-		)
-		(stroke
-			(width 0)
-			(type default)
-		)
-	)
-	(wire
-		(pts
 			(xy 127 86.36) (xy 127 87.63)
 		)
@@
 		(pts
 			(xy 115.57 110.49) (xy 115.57 111.76)
+		)
+		(stroke
+			(width 0)
+			(type default)
+		)
+	)
+	(wire
+		(pts
+			(xy 119.38 77.47) (xy 127 77.47)
 		)
 		(stroke
@@
 	)
 	(label "RXD"
-		(at 119.38 82.55 0)
-		(effects
-			(font
+		(at 119.38 77.47 0)
+		(effects
+			(font
